File: cm5testcarrier.kicad_sch (KiCad schematic)
At the start: 24 parts, among them J1 Barrel_Jack, J2 Conn_02x20_Odd_Even, J3 USB_A, J4 Micro_SD_Card_Det2, U1 MagJack-A70-112-331N126, U2 TPS56A37RPAR

Commit message: Added USB 3.0 ports & added VBUS current reg
Found a newer version of the USB current limiter so I implemented that.
Added USB 3.0 ports and reorganized some nets a bit
Parts:
- added C2, C5, C6: 10u, Capacitor_SMD:C_0805_2012Metric, symbol Device:C
- added C4: 100uF, Capacitor_Tantalum_SMD:CP_EIA-7343-31_Kemet-D, symbol Device:C_Polarized
- added J5: USB3_A, CM5IO:MTCONN_UBAF30-D2011, symbol CM5IO:USB3_A
- added R4: 10k 1%, symbol Device:R
- added U3: AP22653W6-7, AP22653W6-7:SOT95P280X145-6N, symbol AP22653W6-7:AP22653W6-7
- renumbered Cboot to Cboot1, Cff to Cff1, Cin to Cin2, Cout to Cout2, Css to Css1, Rfbb to Rfbb1, Rfbt to Rfbt1, Rmode to Rmode1, Rpg to Rpg1
Connections:
- net +5V: now also C2.2, U3.1 (IN); no longer J3.1 (VBUS)
- net GND: now also C2.1, C4.1, C5.1, C6.1, J5.10 (SHIELD), J5.A4 (GND), J5.A7 (DRAIN), J5.B4 (GND), J5.B7 (DRAIN), R4.2, U3.2 (GND)
- net VBUS_EN: now reaches Module1.111 (VBUS_EN)
- net VBUS_EN: now also U3.3 (EN)
- net USB3-0-RX_N: now reaches Module1.128 (USB3-0-RX_N)
- net USB3-0-RX_N: now also J5.A6 (SSRX+)
- net USB3-0-RX_P: now reaches Module1.130 (USB3-0-RX_P)
- net USB3-0-RX_P: now also J5.A5 (SSRX-)
- net USB3-0-D_P: now reaches Module1.134 (USB3-0-D_P)
- net USB3-0-D_P: now also J5.A3 (D+)
- net USB3-0-D_N: now reaches Module1.136 (USB3-0-D_N)
- net USB3-0-D_N: now also J5.A2 (D-)
- net USB3-0-TX_N: now reaches Module1.140 (USB3-0-TX_N)
- net USB3-0-TX_N: now also J5.A9 (SSTX+)
- net USB3-0-TX_P: now reaches Module1.142 (USB3-0-TX_P)
- net USB3-0-TX_P: now also J5.A8 (SSTX-)
- net USB3-1-RX_N: now reaches Module1.157 (USB3-1-RX_N)
- net USB3-1-RX_N: now also J5.B6 (SSRX+)
- net USB3-1-RX_P: now reaches Module1.159 (USB3-1-RX_P)
- net USB3-1-RX_P: now also J5.B5 (SSRX-)
- net USB3-1-D_P: now reaches Module1.163 (USB3-1-D_P)
- net USB3-1-D_P: now also J5.B3 (D+)
- net USB3-1-D_N: now reaches Module1.165 (USB3-1-D_N)
- net USB3-1-D_N: now also J5.B2 (D-)
- net USB3-1-TX_N: now reaches Module1.169 (USB3-1-TX_N)
- net USB3-1-TX_N: now also J5.B9 (SSTX+)
- net USB3-1-TX_P: now reaches Module1.171 (USB3-1-TX_P)
- net USB3-1-TX_P: now also J5.B8 (SSTX-)
- new net: R4.1, U3.5 (ILIM)
- new net VBUS: C4.2, C5.2, C6.2, J3.1 (VBUS), J5.A1 (VBUS), J5.B1 (VBUS), U3.6 (OUT)
- no-connect marks 0 -> 1
Other:
- note added: "Current Limit switch"
- note added: "USB 2.0 x1"
- note added: "USB 3.0 x2"
- note removed: "USB 2"
- moved on the sheet: J3

Commit message: Servo Controller Finished miscs things reorganized
 - implemented Servo Controller
 - split servo voltage supplies
 - corrected gpio connections
 - implemented fan connector
 - made the usb 2.0 more tidy
 - cleaned up pin nets
Parts:
- added C3: 10u, Capacitor_SMD:C_0805_2012Metric, symbol Device:C
- added C7: 10uF, Capacitor_SMD:C_0805_2012Metric, symbol Device:C
- added Fan_Header1: Conn_01x04_Pin, symbol Connector:Conn_01x04_Pin
- added R5, R6, R7: 10K, Resistor_SMD:R_0402_1005Metric, symbol Adafruit PCA9685 rev C-eagle-import:RESISTOR0805_NOOUTLINE
- added R8: 10K 1%, symbol Device:R
- added RN1, RN2, RN3, RN4: 220, 220 ohm resistor net CAY16:BO_CAY16-L, symbol Device:R_Pack04_SIP_Split
- added SERVO_0-3, SERVO_12-15, SERVO_4-7, SERVO_8-11: HEADER-3X04, 12pin header:CON12_3X4_TU_TSW_SAI, symbol Adafruit PCA9685 rev C-eagle-import:HEADER-3X04
- added U4: PCA9685, PCA9685:TSSOP28_SOT361-1_NXP-L, symbol Adafruit PCA9685 rev C-eagle-import:PCA9685
- AP22653W6-7: renamed from U3; value AP22653W6-7 -> U3; footprint AP22653W6-7:SOT95P280X145-6N -> AP22653W6_7 USB curernt limit switch:SOT95P280X145-6N
- C4: footprint Capacitor_Tantalum_SMD:CP_EIA-7343-31_Kemet-D -> Capacitor_SMD:C_0805_2012Metric
- Cboot1, Cff1, Cin1, Cin2, Cout1, Cout2, Css1: footprint (none) -> Capacitor_SMD:C_0805_2012Metric
- L1: footprint (none) -> Inductor_SMD:L_0402_1005Metric
- Power_LED1: renamed from D2; value LED Red -> D2
- R4, Rfbb1, Rfbt1, Rmode1, Rpg1: footprint (none) -> Resistor_SMD:R_0402_1005Metric
- SD_Card_Reader1: renamed from J4; footprint (none) -> CM5IO:SDCARD_MOLEX_503398-1892
- TPS56A37RPAR1: renamed from U2; footprint RPA0010A-MFG -> TPS56A37:RPA0010A-MFG
- USB2_A1: renamed from J3; value USB_A -> J2; footprint (none) -> Connector_USB:USB_A_Molex_67643_Horizontal
- USB3_A*2: renamed from J5; value USB3_A -> J3
- renumbered J1 to Barrel_Jack1, U1 to Ethernet_Jack1, J2 to GPIO1
Connections:
- net +3V3: now also Module1.78 (GPIO_VREF(1.8v/3.3v_Input)), R8.2
- net +5V: now also C7.2, Fan_Header1.1 (Pin_1), R5.1, R6.1, U4.28 (VDD)
- net GND: now also SD_Card_Reader1.11 (SHIELD), SD_Card_Reader1.6 (VSS), C3.2, C7.1, Fan_Header1.3 (Pin_3), R7.1, SERVO_0-3.12, SERVO_0-3.3, SERVO_0-3.6, SERVO_0-3.9, SERVO_12-15.12, SERVO_12-15.3, SERVO_12-15.6, SERVO_12-15.9, SERVO_4-7.12, SERVO_4-7.3, SERVO_4-7.6, SERVO_4-7.9, SERVO_8-11.12, SERVO_8-11.3, SERVO_8-11.6, SERVO_8-11.9, U4.14 (GND), U4.25 (EXTCLK)
- net GPIO0: now also Module1.36 (ID_SD)
- net GPIO1: now also Module1.35 (ID_SC)
- net USB3-0-RX_N: no longer Module1.128 (USB3-0-RX_N)
- net FAN_TACHOMETER: now reaches Module1.16 (FAN_TACHO)
- net FAN_TACHOMETER: now also Fan_Header1.4 (Pin_4)
- net FAN_PWM: now reaches Module1.19 (FAN_PWM)
- net FAN_PWM: now also Fan_Header1.2 (Pin_2), R8.1
- net SD_CLK: now reaches Module1.57 (SD_CLK)
- net SD_CLK: now also SD_Card_Reader1.5 (CLK)
- net SD_DAT3: now reaches Module1.61 (SD_DAT3)
- net SD_DAT3: now also SD_Card_Reader1.2 (DAT3/CD)
- net SD_DAT0: now reaches Module1.63 (SD_DAT0)
- net SD_DAT0: now also SD_Card_Reader1.7 (DAT0)
- net SD_DAT1: now reaches Module1.67 (SD_DAT1)
- net SD_DAT1: now also SD_Card_Reader1.8 (DAT1)
- net SD_DAT2: now reaches Module1.69 (SD_DAT2)
- net SD_DAT2: now also SD_Card_Reader1.1 (DAT2)
- net SD_PWR_ON: now reaches Module1.75 (SD_PWR_ON)
- net PCA_SCL: now reaches Module1.80 (SCL0)
- net PCA_SCL: now also R6.2, U4.26 (SCL)
- net PCA_SDA: now reaches Module1.82 (SDA0)
- net PCA_SDA: now also R5.2, U4.27 (SDA)
- net SD_CMD: now reaches SD_Card_Reader1.3 (CMD)
- net SD_PWR: now reaches SD_Card_Reader1.4 (VDD)
- net SD_PWR: now also C3.1
- new net: RN4.1 (R1.1), SERVO_12-15.1
- new net: RN1.3 (R2.1), SERVO_0-3.4
- new net: RN1.1 (R1.1), SERVO_0-3.1
- new net: RN1.7 (R4.1), SERVO_0-3.10
- new net: SERVO_0-3.11, SERVO_0-3.2, SERVO_0-3.5, SERVO_0-3.8, SERVO_4-7.11, SERVO_4-7.2, SERVO_4-7.5, SERVO_4-7.8
- new net: RN1.5 (R3.1), SERVO_0-3.7
- new net: RN4.5 (R3.1), SERVO_12-15.7
- new net: RN3.5 (R3.1), SERVO_8-11.7
- new net: RN2.3 (R2.1), SERVO_4-7.4
- new net: RN4.3 (R2.1), SERVO_12-15.4
- new net: RN2.7 (R4.1), SERVO_4-7.10
- new net: RN3.1 (R1.1), SERVO_8-11.1
- new net: RN2.1 (R1.1), SERVO_4-7.1
- new net: RN2.5 (R3.1), SERVO_4-7.7
- new net: RN4.7 (R4.1), SERVO_12-15.10
- new net: SERVO_12-15.11, SERVO_12-15.2, SERVO_12-15.5, SERVO_12-15.8, SERVO_8-11.11, SERVO_8-11.2, SERVO_8-11.5, SERVO_8-11.8
- new net: R7.2, U4.23 (#OE)
- new net: RN3.3 (R2.1), SERVO_8-11.4
- new net: RN3.7 (R4.1), SERVO_8-11.10
- new net Servo_PWM_0: RN1.2 (R1.2), U4.6 (PWM0)
- new net Servo_PWM_1: RN1.4 (R2.2), U4.7 (PWM1)
- new net Servo_PWM_10: RN3.6 (R3.2), U4.17 (PWM10)
- new net Servo_PWM_11: RN3.8 (R4.2), U4.18 (PWM11)
- new net Servo_PWM_12: RN4.2 (R1.2), U4.19 (PWM12)
- new net Servo_PWM_13: RN4.4 (R2.2), U4.20 (PWM13)
- new net Servo_PWM_14: RN4.6 (R3.2), U4.21 (PWM14)
- new net Servo_PWM_15: RN4.8 (R4.2), U4.22 (PWM15)
- new net Servo_PWM_2: RN1.6 (R3.2), U4.8 (PWM2)
- new net Servo_PWM_3: RN1.8 (R4.2), U4.9 (PWM3)
- new net Servo_PWM_4: RN2.2 (R1.2), U4.10 (PWM4)
- new net Servo_PWM_5: RN2.4 (R2.2), U4.11 (PWM5)
- new net Servo_PWM_6: RN2.6 (R3.2), U4.12 (PWM6)
- new net Servo_PWM_7: RN2.8 (R4.2), U4.13 (PWM7)
- new net Servo_PWM_8: RN3.2 (R1.2), U4.15 (PWM8)
- new net Servo_PWM_9: RN3.4 (R2.2), U4.16 (PWM9)
- no-connect marks 1 -> 9
Other:
- note added: "Address: 0x40"
- note added: "Fan Connector"
- note added: "Left CM5 Pin header"
- note added: "PWM Controller"
- note added: "Right CM5 Pin header"
- note added: "SD Boot"
- note added: "Unused 12c address registers"
- note added: "servo jumper connectors"
- note removed: "Power LED"
- moved on the sheet: Barrel_Jack1, GPIO1, Power_LED1, R3

Commit message: Updated footprints & reorganized file structure
 - changed footprints to hand solderable sizes
 - made the file structure make more sense
 - removed files that were not needed in the project
Parts:
- removed Barrel_Jack1: Barrel_Jack, Connector_BarrelJack:BarrelJack_CUI_PJ-063AH_Horizontal, symbol Connector:Barrel_Jack
- removed Cboot1, Cff1: 150 pF, Capacitor_SMD:C_0805_2012Metric, symbol Device:C
- removed Cin1, Cin2: 10uf, Capacitor_SMD:C_0805_2012Metric, symbol Device:C
- removed Cout1, Cout2, Css1: 22 nF, Capacitor_SMD:C_0805_2012Metric, symbol Device:C
- removed L1: 3.3 µH, Inductor_SMD:L_0402_1005Metric, symbol Device:L
- removed Rfbb1: 10 kΩ, Resistor_SMD:R_0402_1005Metric, symbol Device:R
- removed Rfbt1: 73.2 kΩ, Resistor_SMD:R_0402_1005Metric, symbol Device:R
- removed Rmode1: 52.3 kΩ, Resistor_SMD:R_0402_1005Metric, symbol Device:R
- removed Rpg1: 100kΩ, Resistor_SMD:R_0402_1005Metric, symbol Device:R
- removed TPS56A37RPAR1: TPS56A37RPAR, TPS56A37:RPA0010A-MFG, symbol 2025-10-21_03-43-26:TPS56A37RPAR
- added D2: Act_Led1, LED_SMD:LED_1206_3216Metric_Pad1.42x1.75mm_HandSolder, symbol Device:LED
- added H1, H2, H3, H4: M3, MountingHole:MountingHole_3.2mm_M3, symbol Mechanical:MountingHole
- added J1: Disable Bluetooth/Wifi, Connector_PinHeader_2.54mm:PinHeader_2x02_P2.54mm_Vertical, symbol Connector_Generic:Conn_02x02_Odd_Even
- added J6: Wago connector, RoboSubCompute.footprints:CONN2_2091-1372_WAGO, symbol WAGO_Conn_2091_1372:2091-1372
- added J7, J8: Wago Connector, RoboSubCompute.footprints:CONN2_2091-1372_WAGO, symbol WAGO_Conn_2091_1372:2091-1372
- added R9: 1k, Resistor_SMD:R_1210_3225Metric_Pad1.30x2.65mm_HandSolder, symbol Device:R
- C1: footprint Capacitor_SMD:C_0402_1005Metric -> Capacitor_SMD:C_1210_3225Metric_Pad1.33x2.70mm_HandSolder
- C2, C3, C4, C5, C6, C7: footprint Capacitor_SMD:C_0805_2012Metric -> Capacitor_SMD:C_1210_3225Metric_Pad1.33x2.70mm_HandSolder
- D1: renamed from Power_LED1; value D2 -> Pow_LED1; footprint LED_SMD:LED_0603_1608Metric -> LED_SMD:LED_1206_3216Metric_Pad1.42x1.75mm_HandSolder
- J10: renamed from SERVO_4-7; footprint 12pin header:CON12_3X4_TU_TSW_SAI -> RoboSubCompute.footprints:CON12_3X4_TU_TSW_SAI
- J11: renamed from SERVO_12-15; footprint 12pin header:CON12_3X4_TU_TSW_SAI -> RoboSubCompute.footprints:CON12_3X4_TU_TSW_SAI
- J12: renamed from SERVO_8-11; footprint 12pin header:CON12_3X4_TU_TSW_SAI -> RoboSubCompute.footprints:CON12_3X4_TU_TSW_SAI
- J2: renamed from USB2_A1; value J2 -> USB2_A1
- J3: renamed from Ethernet_Jack1; footprint CM5IO:TRJG0926HENL -> Connector_RJ:RJ45_Amphenol_54602-x08_Horizontal
- J3: renamed from USB3_A*2; value J3 -> USB3_A*2; footprint CM5IO:MTCONN_UBAF30-D2011 -> Connector_RJ:RJ45_Amphenol_54602-x08_Horizontal
- J4: renamed from SD_Card_Reader1; footprint CM5IO:SDCARD_MOLEX_503398-1892 -> RoboSubCompute.footprints:SDCARD_MOLEX_503398-1892
- J5: renamed from Fan_Header1; value Conn_01x04_Pin -> Fan_Header; footprint (none) -> Connector:FanPinHeader_1x04_P2.54mm_Vertical
- J9: renamed from SERVO_0-3; footprint 12pin header:CON12_3X4_TU_TSW_SAI -> RoboSubCompute.footprints:CON12_3X4_TU_TSW_SAI
- Module1: footprint CM5IO:Raspberry-Pi-5-Compute-Module -> RoboSubCompute.footprints:Raspberry-Pi-5-Compute-Module; digikey pn (none) -> 609-10164227-1001A1RLFCT-ND
- R1, R2: value 470R -> 470; footprint Resistor_SMD:R_0402_1005Metric -> Resistor_SMD:R_1210_3225Metric_Pad1.30x2.65mm_HandSolder
- R3, R4, R5, R6, R7: footprint Resistor_SMD:R_0402_1005Metric -> Resistor_SMD:R_1210_3225Metric_Pad1.30x2.65mm_HandSolder
- R8: footprint (none) -> Resistor_SMD:R_1210_3225Metric_Pad1.30x2.65mm_HandSolder
- RN1, RN2, RN3, RN4: footprint 220 ohm resistor net CAY16:BO_CAY16-L -> RoboSubCompute.footprints:4x_220_resistor_net
- U3: renamed from AP22653W6-7; value U3 -> AP22653W6-7; footprint AP22653W6_7 USB curernt limit switch:SOT95P280X145-6N -> RoboSubCompute.footprints:USB_Current_limit_Switch_AP22653W6-7
- U4: value PCA9685 -> PCA9685PW,118; footprint PCA9685:TSSOP28_SOT361-1_NXP-L -> RoboSubCompute.footprints:servo_controller_pca9685; DigiKey_PN (none) -> 568-11925-1-ND
- renumbered GPIO1 to J13
Connections:
- net +3V3: now also D2.2 (A)
- net +5V: now also J6.1
- net GND: now also Module1.113 (GND), Module1.59 (GND), J1.2 (Pin_2), J1.4 (Pin_4), J6.2, J7.2, J8.2
- net +Servo 0-7 voltage: now reaches J10.11, J10.2, J10.5, J10.8, J9.11, J9.2, J9.5, J9.8
- net +Servo 0-7 voltage: now also J7.1
- net Act_LED: now reaches Module1.21 (LED_nACT)
- net Act_LED: now also R9.1
- net Disable_wifi: now reaches Module1.89 (WiFi_nDisable)
- net Disable_wifi: now also J1.3 (Pin_3)
- net Disable_bt: now reaches Module1.91 (BT_nDisable)
- net Disable_bt: now also J1.1 (Pin_1)
- net Power_LED: now reaches Module1.95 (LED_nPWR), R3.1
- net +Servo 8-15 voltage: now reaches J11.11, J11.2, J11.5, J11.8, J12.11, J12.2, J12.5, J12.8
- net +Servo 8-15 voltage: now also J8.1
- new net: D2.1 (K), R9.2
- no-connect marks 9 -> 74
Other:
- note added: "DC inputs"
- note removed: "12vdc -> 5vdc"
- note removed: "Buck Converter"
- moved on the sheet: D1, J5, R3, R7, R8

Commit message: Add CSI connector footprint, symbol, and model
 - Partially routed USB 3.0
 - routed ethernet
 - added LEDs
 - updated BOM
 - switched passives to 0805 to save space
 - added CSI/DSI ports (still unrouted)
 - adjusted placement of ports
 - updated README w/ more detailed descriptions
Parts:
- removed D1: Pow_LED1, LED_SMD:LED_1206_3216Metric_Pad1.42x1.75mm_HandSolder, symbol Device:LED
- removed D2: Act_Led1, LED_SMD:LED_1206_3216Metric_Pad1.42x1.75mm_HandSolder, symbol Device:LED
- removed J2: USB2_A1, Connector_USB:USB_A_Molex_67643_Horizontal, symbol Connector:USB_A
- removed J3: MagJack-A70-112-331N126, Connector_RJ:RJ45_Amphenol_54602-x08_Horizontal, symbol CM5IO:MagJack-A70-112-331N126
- removed J3: USB3_A*2, Connector_RJ:RJ45_Amphenol_54602-x08_Horizontal, symbol CM5IO:USB3_A
- removed J4: Micro_SD_Card_Det2, RoboSubCompute.footprints:SDCARD_MOLEX_503398-1892, symbol Connector:Micro_SD_Card_Det2
- added Act_LED1: 150120GS75000, SamacSys_Parts:LEDC3214X68N, symbol SamacSys_Parts:150120GS75000
- added J14: GSB3112311HR, SamacSys_Parts:GSB3112311HR, symbol SamacSys_Parts:GSB3112311HR
- added J16, J17: TF38-22S-0.5SV_830_, SamacSys_Parts:TF3822S05SV830, symbol SamacSys_Parts:TF38-22S-0.5SV_830_
- added J2: GSB191217FHR, GSB191217FHR, symbol SamacSys_Parts:GSB191217FHR
- added J3: ARJM11B1-502-NN-EW2, ARJM11B1502NNEW2, symbol SamacSys_Parts:ARJM11B1-502-NN-EW2
- added J4: GTFP08432B1HR, SamacSys_Parts:GTFP08432B1HR, symbol SamacSys_Parts:GTFP08432B1HR
- added Pwr_Led1: 150120RS75000, SamacSys_Parts:LEDC3216X68N, symbol SamacSys_Parts:150120RS75000
- added R10: 10K, Resistor_SMD:R_0805_2012Metric_Pad1.20x1.40mm_HandSolder, symbol Device:R
- added R11: 2.2K, SamacSys_Parts:ERJS06_U06__0805_, symbol Device:R
- added U2: RT9742GGJ5, SamacSys_Parts:SOT94P280X100-5N, symbol CM5IO:RT9742GGJ5
- C1: value 100n -> 100p; footprint Capacitor_SMD:C_1210_3225Metric_Pad1.33x2.70mm_HandSolder -> Capacitor_SMD:C_0805_2012Metric_Pad1.18x1.45mm_HandSolder; Mouser Part Number (none) -> 581-08055C101K
- C2, C3, C5, C6: footprint Capacitor_SMD:C_1210_3225Metric_Pad1.33x2.70mm_HandSolder -> Capacitor_SMD:C_0805_2012Metric_Pad1.18x1.45mm_HandSolder; Mouser Part Number (none) -> 581-08056D106K
- C4: value 100uF -> 100u; footprint Capacitor_SMD:C_1210_3225Metric_Pad1.33x2.70mm_HandSolder -> Capacitor_SMD:C_0805_2012Metric_Pad1.18x1.45mm_HandSolder; Mouser Part Number (none) -> 963-JMK325BJ107MM-T
- C7: value 10uF -> 10u; footprint Capacitor_SMD:C_1210_3225Metric_Pad1.33x2.70mm_HandSolder -> Capacitor_SMD:C_0805_2012Metric_Pad1.18x1.45mm_HandSolder; Mouser Part Number (none) -> 581-08056D106K
- J13: Mouser Part Number (none) -> 798-FH12-22S-0.5SH55
- J6: value Wago connector -> Wago connector 2091-1372; Mouser Part Number (none) -> DigiKey
- J7, J8: value Wago Connector -> Wago connector 2091-1372; Mouser Part Number (none) -> DigiKey
- Module1: Mouser Part Number (none) -> 649-01642271001A1RLF; digikey pn 609-10164227-1001A1RLFCT-ND -> (none)
- R1, R2: value 470 -> 2.2K; footprint Resistor_SMD:R_1210_3225Metric_Pad1.30x2.65mm_HandSolder -> SamacSys_Parts:ERJS06_U06__0805_; Mouser Part Number (none) -> 667-ERJ-U06D2201V
- R3: value 1k -> 150; footprint Resistor_SMD:R_1210_3225Metric_Pad1.30x2.65mm_HandSolder -> Resistor_SMD:R_0805_2012Metric_Pad1.20x1.40mm_HandSolder; Mouser Part Number (none) -> 667-ERJ-UP6D1500V
- R4: value 10k 1% -> 10k; footprint Resistor_SMD:R_1210_3225Metric_Pad1.30x2.65mm_HandSolder -> Resistor_SMD:R_0805_2012Metric_Pad1.20x1.40mm_HandSolder; Mouser Part Number (none) -> 667-ERJ-UP6D1002V
- R5, R6, R7: footprint Resistor_SMD:R_1210_3225Metric_Pad1.30x2.65mm_HandSolder -> Resistor_SMD:R_0805_2012Metric_Pad1.20x1.40mm_HandSolder; Mouser Part Number (none) -> 667-ERJ-UP6D1002V
- R8: value 10K 1% -> 10K; footprint Resistor_SMD:R_1210_3225Metric_Pad1.30x2.65mm_HandSolder -> Resistor_SMD:R_0805_2012Metric_Pad1.20x1.40mm_HandSolder; Mouser Part Number (none) -> 667-ERJ-UP6D1002V
- R9: value 1k -> 90; footprint Resistor_SMD:R_1210_3225Metric_Pad1.30x2.65mm_HandSolder -> Resistor_SMD:R_0805_2012Metric_Pad1.20x1.40mm_HandSolder; Mouser Part Number (none) -> 667-ERJ-UP6D91R0V
- RN1, RN2, RN3, RN4: footprint RoboSubCompute.footprints:4x_220_resistor_net -> SamacSys_Parts:CAT161000F4; Mouser Part Number (none) -> 652-CAT16-2200F4LF
- U3: footprint RoboSubCompute.footprints:USB_Current_limit_Switch_AP22653W6-7 -> SamacSys_Parts:SOT95P280X145-6N; Mouser Part Number (none) -> 621-AP22653W6-7
- U4: footprint RoboSubCompute.footprints:servo_controller_pca9685 -> SamacSys_Parts:SOP65P640X110-28N; DigiKey_PN 568-11925-1-ND -> (none); Mouser Part Number (none) -> 771-PCA9685PW,118
Connections:
- net +3V3: now also R1.2, R2.2, Act_LED1.2 (A), J16.22, J17.22, R11.2
- net +5V: now also Pwr_Led1.2 (A)
- net GND: now also J14.13 (GND_2), J14.16 (GND_DRAIN_2), J14.19 (SHIELD_1), J14.20 (SHIELD_2), J14.21 (SHIELD_3), J14.22 (SHIELD_4), J14.4 (GND_1), J14.7 (GND_DRAIN_1), J16.1, J16.10, J16.13, J16.16, J16.19, J16.4, J16.7, J16.MP1, J16.MP2, J16.MP3, J16.MP4, J17.1, J17.10, J17.13, J17.16, J17.19, J17.4, J17.7, J17.MP1, J17.MP2, J17.MP3, J17.MP4, J2.4 (GND), J2.MH1, J2.MH2, J2.MH3, J2.MH4, J3.13 (MH_1), J3.14 (MH_2), J4.10 (GROUND_1), J4.11 (GROUND_2), J4.12 (GROUND_3), J4.6 (VSS), U2.2 (GND)
- net GPIO0: now also J16.21, R11.1
- net GPIO1: now also R2.1, J16.20
- net GPIO2: now also R5.2, U4.27 (SDA)
- net GPIO3: now also R6.2, U4.26 (SCL)
- net SD_CLK: now also J4.5 (CLK)
- net SD_CMD: now also Module1.62 (SD_CMD), J4.3 (CMD)
- net SD_DAT0: now also J4.7 (DAT0)
- net SD_DAT1: now also J4.8 (DAT1)
- net SD_DAT2: now also J4.1 (DAT2)
- net SD_DAT3: now also J4.2 (CD/DAT3)
- net SD_PWR: now also J4.4 (VDD), U2.1 (OUT)
- net SD_PWR_ON: now also R10.2, U2.4 (EN)
- net USB3-0-D_N: now also J14.2 (D-_1)
- net USB3-0-D_P: now also J14.3 (D+_1)
- net USB3-0-RX_N: now also Module1.128 (USB3-0-RX_N), J14.5 (SSRX-_1)
- net USB3-0-RX_P: now also J14.6 (SSRX+_1)
- net USB3-0-TX_N: now also J14.8 (SSTX-_1)
- net USB3-0-TX_P: now also J14.9 (SSTX+_1)
- net USB3-1-D_N: now also J14.11 (D-_2)
- net USB3-1-D_P: now also J14.12 (D+_2)
- net USB3-1-RX_N: now also J14.14 (SSRX-_2)
- net USB3-1-RX_P: now also J14.15 (SSRX+_2)
- net USB3-1-TX_N: now also J14.17 (SSTX-_2)
- net USB3-1-TX_P: now also J14.18 (SSTX+_2)
- net USB_2_N: now also J2.2 (D-)
- net USB_2_P: now also J2.3 (D+)
- net VBUS: now also J14.1 (VBUS_1), J14.10 (VBUS_2), J2.1 (VBUS)
- net p+0: now also J3.1 (TD1+)
- net p+1: now also Module1.4 (Ethernet_Pair1_P), J3.3 (TD2+)
- net p+2: now also J3.7 (TD3+); no longer Module1.4 (Ethernet_Pair1_P)
- net p+3: now also J3.9 (TD4+)
- net p-0: now also J3.2 (TD1-)
- net p-1: now also J3.4 (TD2-)
- net p-2: now also J3.8 (TD3-)
- net p-3: now also J3.10 (TD4-)
- net at R1.1: now also J16.17
- net at C1.2: now also J3.5 (CT_1), J3.6 (CT_2)
- net at R9.2: now also Act_LED1.1 (K)
- net CAM_GPIO1: now reaches Module1.100 (CAM_GPIO1)
- net CAM_GPIO1: now also J17.18
- net CAM_GPIO0: now reaches Module1.97 (CAM_GPIO0)
- net CAM_GPIO0: now also J17.17
- net at R3.2: now also Pwr_Led1.1 (K)
- net DPHY0_D0_N: now reaches Module1.115 (MIPI0_D0_N)
- net DPHY0_D0_N: now also J17.2
- net DPHY0_D0_P: now reaches Module1.117 (MIPI0_D0_P)
- net DPHY0_D0_P: now also J17.3
- net DPHY0_D1_N: now reaches Module1.121 (MIPI0_D1_N)
- net DPHY0_D1_N: now also J17.5
- net DPHY0_D1_P: now reaches Module1.123 (MIPI0_D1_P)
- net DPHY0_D1_P: now also J17.6
- net DPHY0_C_N: now reaches Module1.127 (MIPI0_C_N)
- net DPHY0_C_N: now also J17.8
- net DPHY0_C_P: now reaches Module1.129 (MIPI0_C_P)
- net DPHY0_C_P: now also J17.9
- net DPHY0_D2_N: now reaches Module1.133 (MIPI0_D2_N)
- net DPHY0_D2_N: now also J17.11
- net DPHY0_D2_P: now reaches Module1.135 (MIPI0_D2_P)
- net DPHY0_D2_P: now also J17.12
- net DPHY0_D3_N: now reaches Module1.139 (MIPI0_D3_N)
- net DPHY0_D3_N: now also J17.14
- net DPHY0_D3_P: now reaches Module1.141 (MIPI0_D3_P)
- net DPHY0_D3_P: now also J17.15
- net DPHY1_D0_N: now reaches Module1.175 (MIPI1_D0_N)
- net DPHY1_D0_N: now also J16.2
- net DPHY1_D0_P: now reaches Module1.177 (MIPI1_D0_P)
- net DPHY1_D0_P: now also J16.3
- net DPHY1_D1_N: now reaches Module1.181 (MIPI1_D1_N)
- net DPHY1_D1_N: now also J16.5
- net DPHY1_D1_P: now reaches Module1.183 (MIPI1_D1_P)
- net DPHY1_D1_P: now also J16.6
- net DPHY1_C_N: now reaches Module1.187 (MIPI1_C_N)
- net DPHY1_C_N: now also J16.8
- net DPHY1_C_P: now reaches Module1.189 (MIPI1_C_P)
- net DPHY1_C_P: now also J16.9
- net DPHY1_D2_N: now reaches Module1.193 (MIPI1_D2_N)
- net DPHY1_D2_N: now also J16.11
- net DPHY1_D3_N: now reaches Module1.194 (MIPI1_D3_N)
- net DPHY1_D3_N: now also J16.14
- net DPHY1_D2_P: now reaches Module1.195 (MIPI1_D2_P)
- net DPHY1_D2_P: now also J16.12
- net DPHY1_D3_P: now reaches Module1.196 (MIPI1_D3_P)
- net DPHY1_D3_P: now also J16.15
- removed net PCA_SCL: Module1.80 (SCL0), R6.2, U4.26 (SCL)
- removed net PCA_SDA: Module1.82 (SDA0), R5.2, U4.27 (SDA)
- net led1: no longer names the net of Module1.15 (Ethernet_nLED3(3.3v))
- net led1: no longer R1.2
- net led2: no longer names the net of Module1.17 (Ethernet_nLED2(3.3v))
- net led2: no longer R2.2
- new net +3.3v: R10.1, U2.5 (IN)
- new net SCL0: J17.20, Module1.80 (SCL0)
- new net SDA0: J17.21, Module1.82 (SDA0)
- no-connect marks 74 -> 60
Other:
- note added: "CSI Connectors"
- note added: "pin name mistmatch ;("
- note removed: "Ethernet"
- company: (none) -> RoboSub
- title: (none) -> ROV Compute Module 5 Control Board
- moved on the sheet: C1, C2, C3, C4, C5, C6, C7, H1, H2, H3, H4, J1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
