File: UTDRoboSubCompute.kicad_pcb (KiCad board)
At the start: 4 copper layers, 100 x 100.1 mm, 52 parts, among them IC1 TPD4E05U06QDQARQ1, IC2 TPD4E05U06QDQARQ1, J1 Disable Bluetooth/Wifi, J10 HEADER-3X04, J11 HEADER-3X04, J12 HEADER-3X04, J13 Conn_02x20_Odd_Even, J14 GSB3116344KHHR, J15 GSB3116344KHHR, J16 TF38-22S-0.5SV_830_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

Commit message: Improve README and update PCB sheet/net refs
Expanded and clarified README: added table of contents, more component details (servo, CSI/DSI, Ethernet, USB, SD boot, power, fan), images, USB config hint (dtoverlay), PCB dimensions, and a recommendation to use the interactive BOM. Updated UTDRoboSubCompute.kicad_pcb: replaced many sheetfile references from cm5testcarrier.kicad_sch to UTDRoboSubCompute.kicad_sch, ), adjusted a pad reference, and refreshed numerous footprint UUIDs. These changes align documentation with the board files and fix net/sheet references used by the PCB and BOM generation.
Parts:
- renumbered Act to Act_LED1, Pwr to Pwr_Led1
Connections:
- Module1 pad 76: unconnected-(Module1A-VBAT-Pad76) -> /VBAT
Routing:
- net /VBUS: track 61.8 -> 65.0 mm
Changed lines of the file:
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@@
 	(net 118 "unconnected-(U3-~{FAULT}-Pad4)")
 	(net 119 "unconnected-(Module1B-HDMI1_TX2_N-Pad148)")
-	(net 120 "unconnected-(Module1A-VBAT-Pad76)")
+	(net 120 "/VBAT")
 	(net 121 "/DPHY0_C_N")
 	(net 122 "/SD_PWR_ON")
@@
 		(property ki_fp_filters "CONN2_2091-1372_WAG")
 		(sheetname "/")
-		(sheetfile "cm5testcarrier.kicad_sch")
+		(sheetfile "UTDRoboSubCompute.kicad_sch")
 		(attr through_hole)
 		(fp_line
@@
 		(property ki_fp_filters "R?Array?SIP*")
 		(sheetname "/")
-		(sheetfile "cm5testcarrier.kicad_sch")
+		(sheetfile "UTDRoboSubCompute.kicad_sch")
 		(attr smd)
 		(fp_line
@@
 		(property ki_fp_filters "C_*")
 		(sheetname "/")
-		(sheetfile "cm5testcarrier.kicad_sch")
+		(sheetfile "UTDRoboSubCompute.kicad_sch")
 		(attr smd)
 		(fp_line
@@
 		)
 		(sheetname "/")
-		(sheetfile "cm5testcarrier.kicad_sch")
+		(sheetfile "UTDRoboSubCompute.kicad_sch")
 		(attr through_hole)
 		(fp_line
@@
 		(property ki_fp_filters "R_*")
 		(sheetname "/")
-		(sheetfile "cm5testcarrier.kicad_sch")
+		(sheetfile "UTDRoboSubCompute.kicad_sch")
 		(attr smd)
 		(fp_line
@@
 		)
 		(sheetname "/")
-		(sheetfile "cm5testcarrier.kicad_sch")
+		(sheetfile "UTDRoboSubCompute.kicad_sch")
 		(attr smd)
 		(fp_line
@@
 		(property ki_fp_filters "R_*")
 		(sheetname "/")
-		(sheetfile "cm5testcarrier.kicad_sch")
+		(sheetfile "UTDRoboSubCompute.kicad_sch")
 		(attr smd)
 		(fp_line
@@
 		(property ki_fp_filters "C_*")
 		(sheetname "/")
-		(sheetfile "cm5testcarrier.kicad_sch")
+		(sheetfile "UTDRoboSubCompute.kicad_sch")
 		(attr smd)
 		(fp_line
@@
 		)
 		(sheetname "/")
-		(sheetfile "cm5testcarrier.kicad_sch")
+		(sheetfile "UTDRoboSubCompute.kicad_sch")
 		(attr through_hole)
 		(fp_line
@@
 		)
 		(sheetname "/")
-		(sheetfile "cm5testcarrier.kicad_sch")
+		(sheetfile "UTDRoboSubCompute.kicad_sch")
 		(attr smd)
 		(fp_line
@@
 			(size 0.2 0.7)
 			(layers "F.Cu" "F.Mask" "F.Paste")
-			(net 120 "unconnected-(Module1A-VBAT-Pad76)")
+			(net 120 "/VBAT")
 			(pinfunction "VBAT")
-			(pintype "passive+no_connect")
+			(pintype "passive")
 		)
 		(pad "77" smd rect
@@
 		)
 		(sheetname "/")
-		(sheetfile "cm5testcarrier.kicad_sch")
+		(sheetfile "UTDRoboSubCompute.kicad_sch")
 		(attr through_hole)
 		(fp_line
@@
 		)
 		(sheetname "/")
-		(sheetfile "cm5testcarrier.kicad_sch")
+		(sheetfile "UTDRoboSubCompute.kicad_sch")
 		(attr smd)
 		(fp_line
@@
 		)
 		(sheetname "/")
-		(sheetfile "cm5testcarrier.kicad_sch")
+		(sheetfile "UTDRoboSubCompute.kicad_sch")
 		(attr through_hole)
 		(fp_line
@@
 		(property ki_fp_filters "R?Array?SIP*")
 		(sheetname "/")
-		(sheetfile "cm5testcarrier.kicad_sch")
+		(sheetfile "UTDRoboSubCompute.kicad_sch")
 		(attr smd)
 		(fp_line
@@
 		(property ki_fp_filters "CP_*")
 		(sheetname "/")
-		(sheetfile "cm5testcarrier.kicad_sch")
+		(sheetfile "UTDRoboSubCompute.kicad_sch")
 		(attr smd)
 		(fp_line
@@
 		(property ki_fp_filters "CONN2_2091-1372_WAG")
 		(sheetname "/")
-		(sheetfile "cm5testcarrier.kicad_sch")
+		(sheetfile "UTDRoboSubCompute.kicad_sch")
 		(attr through_hole)
 		(fp_line
@@
 		(property ki_fp_filters "R?Array?SIP*")
 		(sheetname "/")
-		(sheetfile "cm5testcarrier.kicad_sch")
+		(sheetfile "UTDRoboSubCompute.kicad_sch")
 		(attr smd)
 		(fp_line
@@
 		(property ki_fp_filters "R_*")
 		(sheetname "/")
-		(sheetfile "cm5testcarrier.kicad_sch")
+		(sheetfile "UTDRoboSubCompute.kicad_sch")
 		(attr smd)
 		(fp_line
@@
 		(property ki_fp_filters "R_*")
 		(sheetname "/")
-		(sheetfile "cm5testcarrier.kicad_sch")
+		(sheetfile "UTDRoboSubCompute.kicad_sch")
 		(attr smd)
 		(fp_circle
@@
 		(property ki_fp_filters "MountingHole*")
 		(sheetname "/")
-		(sheetfile "cm5testcarrier.kicad_sch")
+		(sheetfile "UTDRoboSubCompute.kicad_sch")
 		(attr exclude_from_pos_files exclude_from_bom)
 		(fp_circle
@@
 		)
 		(sheetname "/")
-		(sheetfile "cm5testcarrier.kicad_sch")
+		(sheetfile "UTDRoboSubCompute.kicad_sch")
 		(attr smd)
 		(fp_line
@@
 		(property ki_fp_filters "MountingHole*")
 		(sheetname "/")
-		(sheetfile "cm5testcarrier.kicad_sch")
+		(sheetfile "UTDRoboSubCompute.kicad_sch")
 		(attr exclude_from_pos_files exclude_from_bom)
 		(fp_circle
@@
 		(property ki_fp_filters "R?Array?SIP*")
 		(sheetname "/")
-		(sheetfile "cm5testcarrier.kicad_sch")
+		(sheetfile "UTDRoboSubCompute.kicad_sch")
 		(attr smd)
 		(fp_line
@@
 		)
 		(sheetname "/")
-		(sheetfile "cm5testcarrier.kicad_sch")
+		(sheetfile "UTDRoboSubCompute.kicad_sch")
 		(attr through_hole)
 		(fp_line
@@
 		)
 		(sheetname "/")
-		(sheetfile "cm5testcarrier.kicad_sch")
+		(sheetfile "UTDRoboSubCompute.kicad_sch")
 		(attr smd)
 		(fp_circle
@@
 		(property ki_fp_filters "C_*")
 		(sheetname "/")
-		(sheetfile "cm5testcarrier.kicad_sch")
+		(sheetfile "UTDRoboSubCompute.kicad_sch")
 		(attr smd)
 		(fp_line
@@
 		(property ki_fp_filters "R_*")
 		(sheetname "/")
-		(sheetfile "cm5testcarrier.kicad_sch")
+		(sheetfile "UTDRoboSubCompute.kicad_sch")
 		(attr smd)
 		(fp_line
@@
 		(property ki_fp_filters "C_*")
 		(sheetname "/")
-		(sheetfile "cm5testcarrier.kicad_sch")
+		(sheetfile "UTDRoboSubCompute.kicad_sch")
 		(attr smd)
 		(fp_line
@@
 		(property ki_fp_filters "Connector*:*_2x??_*")
 		(sheetname "/")
-		(sheetfile "cm5testcarrier.kicad_sch")
+		(sheetfile "UTDRoboSubCompute.kicad_sch")
 		(attr through_hole)
 		(fp_line
@@
 		(property ki_fp_filters "C_*")
 		(sheetname "/")
-		(sheetfile "cm5testcarrier.kicad_sch")
+		(sheetfile "UTDRoboSubCompute.kicad_sch")
 		(attr smd)
 		(fp_line
@@
 		(property ki_fp_filters "MountingHole*")
 		(sheetname "/")
-		(sheetfile "cm5testcarrier.kicad_sch")
+		(sheetfile "UTDRoboSubCompute.kicad_sch")
 		(attr exclude_from_pos_files exclude_from_bom)
 		(fp_circle
@@
 		(property ki_fp_filters "Connector*:*_2x??_*")
 		(sheetname "/")
-		(sheetfile "cm5testcarrier.kicad_sch")
+		(sheetfile "UTDRoboSubCompute.kicad_sch")
 		(attr through_hole)
 		(fp_line
@@
 		)
 		(sheetname "/")
-		(sheetfile "cm5testcarrier.kicad_sch")
+		(sheetfile "UTDRoboSubCompute.kicad_sch")
 		(attr through_hole)
 		(fp_line
@@
 		)
 		(sheetname "/")
-		(sheetfile "cm5testcarrier.kicad_sch")
+		(sheetfile "UTDRoboSubCompute.kicad_sch")
 		(attr smd)
 		(fp_circle
@@
 		(property ki_fp_filters "R_*")
 		(sheetname "/")
-		(sheetfile "cm5testcarrier.kicad_sch")
+		(sheetfile "UTDRoboSubCompute.kicad_sch")
 		(attr smd)
 		(fp_line
@@
 		(property ki_fp_filters "CONN2_2091-1372_WAG")
 		(sheetname "/")
-		(sheetfile "cm5testcarrier.kicad_sch")
+		(sheetfile "UTDRoboSubCompute.kicad_sch")
 		(attr through_hole)
 		(fp_line
@@
 		(descr "3016 (1206) _1")
 		(tags "LED")
-		(property "Reference" "Pwr"
+		(property "Reference" "Pwr_Led1"
 			(at 3.97 0.18 0)
 			(layer "F.SilkS")
@@
 		)
 		(sheetname "/")
-		(sheetfile "cm5testcarrier.kicad_sch")
+		(sheetfile "UTDRoboSubCompute.kicad_sch")
 		(attr smd)
 		(fp_line
@@
 		(property ki_fp_filters "R_*")
 		(sheetname "/")
-		(sheetfile "cm5testcarrier.kicad_sch")
+		(sheetfile "UTDRoboSubCompute.kicad_sch")
 		(attr smd)
 		(fp_circle
@@
 		)
 		(sheetname "/")
-		(sheetfile "cm5testcarrier.kicad_sch")
+		(sheetfile "UTDRoboSubCompute.kicad_sch")
 		(attr smd)
 		(fp_line
@@
 		(property ki_fp_filters "C_*")
 		(sheetname "/")
-		(sheetfile "cm5testcarrier.kicad_sch")
+		(sheetfile "UTDRoboSubCompute.kicad_sch")
 		(attr smd)
 		(fp_line
@@
 		)
 		(sheetname "/")
-		(sheetfile "cm5testcarrier.kicad_sch")
+		(sheetfile "UTDRoboSubCompute.kicad_sch")
 		(attr smd)
 		(fp_line
@@
 		)
 		(sheetname "/")
-		(sheetfile "cm5testcarrier.kicad_sch")
+		(sheetfile "UTDRoboSubCompute.kicad_sch")
 		(attr smd)
 		(fp_line
@@
 		(property ki_fp_filters "Connector*:*_1x??_*")
 		(sheetname "/")
-		(sheetfile "cm5testcarrier.kicad_sch")
+		(sheetfile "UTDRoboSubCompute.kicad_sch")
 		(attr through_hole)
 		(fp_line
@@
 		(descr "150120GS75000")
 		(tags "LED")
-		(property "Reference" "Act"
+		(property "Reference" "Act_LED1"
 			(at 3.97 0.1 180)
 			(layer "F.SilkS")
@@
 		)
 		(sheetname "/")
-		(sheetfile "cm5testcarrier.kicad_sch")
+		(sheetfile "UTDRoboSubCompute.kicad_sch")
 		(attr smd)
 		(fp_line
@@
 		)
 		(sheetname "/")
-		(sheetfile "cm5testcarrier.kicad_sch")
+		(sheetfile "UTDRoboSubCompute.kicad_sch")
 		(attr through_hole)
 		(fp_line
@@
 		)
 		(sheetname "/")
-		(sheetfile "cm5testcarrier.kicad_sch")
+		(sheetfile "UTDRoboSubCompute.kicad_sch")
 		(attr smd)
 		(fp_line
@@
 		(property ki_fp_filters "R_*")
 		(sheetname "/")
-		(sheetfile "cm5testcarrier.kicad_sch")
+		(sheetfile "UTDRoboSubCompute.kicad_sch")
 		(attr smd)
 		(fp_circle
@@
 		)
 		(sheetname "/")
-		(sheetfile "cm5testcarrier.kicad_sch")
+		(sheetfile "UTDRoboSubCompute.kicad_sch")
 		(attr smd)
 		(fp_line
@@
 		)
 		(sheetname "/")
-		(sheetfile "cm5testcarrier.kicad_sch")
+		(sheetfile "UTDRoboSubCompute.kicad_sch")
 		(attr through_hole)
 		(fp_line
@@
 		(property ki_fp_filters "MountingHole*")
 		(sheetname "/")
-		(sheetfile "cm5testcarrier.kicad_sch")
+		(sheetfile "UTDRoboSubCompute.kicad_sch")
 		(attr exclude_from_pos_files exclude_from_bom)
 		(fp_circle
@@
 		)
 		(sheetname "/")
-		(sheetfile "cm5testcarrier.kicad_sch")
+		(sheetfile "UTDRoboSubCompute.kicad_sch")
 		(attr smd)
 		(fp_line
@@
 	)
 	(segment
+		(start 174.4 99.9)
+		(end 174.4 103.088933)
+		(width 0.8)
+		(layer "F.Cu")
+		(net 5)
+	)
+	(segment
 		(start 168.9625 102.1)
 		(end 168.9625 104.3)
@@
 		(polygon
 			(pts
-				(xy 95.6 55.1) (xy 95.6 155.3) (xy 196 155.3) (xy 195.820489 65.36475) (xy 195.8 55.1)
+				(xy 194.99 55.1) (xy 95.6 55.1) (xy 95.6 155.3) (xy 196 155.3) (xy 195.820489 65.36475) (xy 195.8 55.1)
 			)
 		)
